Commit message: test

File: description/urdf/coxa_link/coxa_link.xacro (robot description, xacro)
@@ -25,5 +25,5 @@
             <parent link="${parent}" />
             <child link="${prefix}_coxa_link" />
-            <limit lower="0" upper="${M_PI}" effort="50.0"
+            <limit lower="${M_PI}" upper="${M_PI}" effort="50.0"
                 velocity="10.0" />
             <dynamics damping="0.0005" friction="0.1" />

File: description/urdf/femur_link/femur_link.xacro (robot description, xacro)
@@ -26,5 +26,5 @@
             <parent link="${parent}" />
             <child link="${prefix}_femur_link" />
-            <limit lower="0" upper="${M_PI}" effort="50.0"
+            <limit lower="${M_PI}" upper="${M_PI}" effort="50.0"
                 velocity="10.0" />
             <dynamics damping="0.0005" friction="0.1" />

File: description/urdf/robot.urdf (robot description, URDF)
Before this commit: robot robot, 15 links, 14 joints
Links:
- added link BL_end_effector_link, mass 0.001; collision sphere radius=0.01; visual sphere radius=0.01
- added link BR_end_effector_link, mass 0.001; collision sphere radius=0.01; visual sphere radius=0.01
- added link FL_end_effector_link, mass 0.001; collision sphere radius=0.01; visual sphere radius=0.01
- added link FR_end_effector_link, mass 0.001; collision sphere radius=0.01; visual sphere radius=0.01
- link BL_coxa_link: geometry collision mesh filename=package://krsri2025/meshes/collision/coxa.stl; visual mesh filename=package://krsri2025/meshes/visual/coxa.dae
- link BL_femur_link: geometry collision mesh filename=package://krsri2025/meshes/collision/femur.stl; visual mesh filename=package://krsri2025/meshes/visual/femur.dae
- link BL_tibia_link: geometry collision mesh filename=package://krsri2025/meshes/collision/tibia.stl; visual mesh filename=package://krsri2025/meshes/visual/tibia.dae
- link BR_coxa_link: geometry collision mesh filename=package://krsri2025/meshes/collision/coxa.stl; visual mesh filename=package://krsri2025/meshes/visual/coxa.dae
- link BR_femur_link: geometry collision mesh filename=package://krsri2025/meshes/collision/femur.stl; visual mesh filename=package://krsri2025/meshes/visual/femur.dae
- link BR_tibia_link: geometry collision mesh filename=package://krsri2025/meshes/collision/tibia.stl; visual mesh filename=package://krsri2025/meshes/visual/tibia.dae
- link FL_coxa_link: geometry collision mesh filename=package://krsri2025/meshes/collision/coxa.stl; visual mesh filename=package://krsri2025/meshes/visual/coxa.dae
- link FL_femur_link: geometry collision mesh filename=package://krsri2025/meshes/collision/femur.stl; visual mesh filename=package://krsri2025/meshes/visual/femur.dae
- link FL_tibia_link: geometry collision mesh filename=package://krsri2025/meshes/collision/tibia.stl; visual mesh filename=package://krsri2025/meshes/visual/tibia.dae
- link FR_coxa_link: geometry collision mesh filename=package://krsri2025/meshes/collision/coxa.stl; visual mesh filename=package://krsri2025/meshes/visual/coxa.dae
- link FR_femur_link: geometry collision mesh filename=package://krsri2025/meshes/collision/femur.stl; visual mesh filename=package://krsri2025/meshes/visual/femur.dae
- link FR_tibia_link: geometry collision mesh filename=package://krsri2025/meshes/collision/tibia.stl; visual mesh filename=package://krsri2025/meshes/visual/tibia.dae
- link base_link: geometry collision mesh filename=package://krsri2025/meshes/collision/base.stl; visual mesh filename=package://krsri2025/meshes/visual/base.dae
Joints:
- added joint BL_end_effector_joint: type fixed, parent BL_tibia_link, child BL_end_effector_link, origin xyz=0.075 0.16952 -0.02273 rpy=0 0 0
- added joint BR_end_effector_joint: type fixed, parent BR_tibia_link, child BR_end_effector_link, origin xyz=0.075 0.16952 -0.02273 rpy=0 0 0
- added joint FL_end_effector_joint: type fixed, parent FL_tibia_link, child FL_end_effector_link, origin xyz=0.075 0.16952 -0.02273 rpy=0 0 0
- added joint FR_end_effector_joint: type fixed, parent FR_tibia_link, child FR_end_effector_link, origin xyz=0.075 0.16952 -0.02273 rpy=0 0 0
- added joint base_footprint_joint: type fixed, parent base_footprint, child base_link, origin xyz=0 0 0 rpy=0 0 0
- joint BL_coxa_link_joint: limit lower=0 upper=3.14159274 effort=50.0 velocity=10.0 -> lower=3.14159274 upper=3.14159274 effort=50.0 velocity=10.0
- joint BL_femur_link_joint: limit lower=0 upper=3.14159274 effort=50.0 velocity=10.0 -> lower=3.14159274 upper=3.14159274 effort=50.0 velocity=10.0
- joint BL_tibia_link_joint: limit lower=0 upper=3.14159274 effort=50.0 velocity=10.0 -> lower=3.14159274 upper=3.14159274 effort=50.0 velocity=10.0
- joint BR_coxa_link_joint: limit lower=0 upper=3.14159274 effort=50.0 velocity=10.0 -> lower=3.14159274 upper=3.14159274 effort=50.0 velocity=10.0
- joint BR_femur_link_joint: limit lower=0 upper=3.14159274 effort=50.0 velocity=10.0 -> lower=3.14159274 upper=3.14159274 effort=50.0 velocity=10.0
- joint BR_tibia_link_joint: limit lower=0 upper=3.14159274 effort=50.0 velocity=10.0 -> lower=3.14159274 upper=3.14159274 effort=50.0 velocity=10.0
- joint FL_coxa_link_joint: limit lower=0 upper=3.14159274 effort=50.0 velocity=10.0 -> lower=3.14159274 upper=3.14159274 effort=50.0 velocity=10.0
- joint FL_femur_link_joint: limit lower=0 upper=3.14159274 effort=50.0 velocity=10.0 -> lower=3.14159274 upper=3.14159274 effort=50.0 velocity=10.0
- joint FL_tibia_link_joint: limit lower=0 upper=3.14159274 effort=50.0 velocity=10.0 -> lower=3.14159274 upper=3.14159274 effort=50.0 velocity=10.0
- joint FR_coxa_link_joint: limit lower=0 upper=3.14159274 effort=50.0 velocity=10.0 -> lower=3.14159274 upper=3.14159274 effort=50.0 velocity=10.0
- joint FR_femur_link_joint: limit lower=0 upper=3.14159274 effort=50.0 velocity=10.0 -> lower=3.14159274 upper=3.14159274 effort=50.0 velocity=10.0
- joint FR_tibia_link_joint: limit lower=0 upper=3.14159274 effort=50.0 velocity=10.0 -> lower=3.14159274 upper=3.14159274 effort=50.0 velocity=10.0

File: description/urdf/tibia_link/tibia_link.xacro (robot description, xacro)
@@ -26,5 +26,5 @@
             <parent link="${parent}" />
             <child link="${prefix}_tibia_link" />
-            <limit lower="0" upper="${M_PI}" effort="50.0"
+            <limit lower="${M_PI}" upper="${M_PI}" effort="50.0"
                 velocity="10.0" />
             <dynamics damping="0.0005" friction="0.1" />
